File: glider/glider.sch (KiCad schematic (older format))
At the start: 127 parts, among them J1 SENSOR_I2C, J10 CELL, J11 SCH1, J12 IO, J13 SCH2, J14 SCH3, J15 SCH4, J16 SCH5, J17 SCH6, J18 SCH7, J19 Micro_SD_Card, J2 USB_B_Micro, J20 Conn_01x02, J3 NCP_EXT, J4 DEBUG_NAV, J5 DEBUG_NCP, J6 SCH8, J7 GPS_UART, J8 NCP_COM, J9 IMU_SPI, Q1 Q_PMOS_DGS, SW1 NAV_NRST, SW2 NAV_BOOT, SW3 NCP_NRST, SW4 NCP_USER, U1 BGM220P, U10 AP2120N-1.8, U11 FXLA0104, U12 RT6218A, U2 STM32G484RETx, U3 MCP1812, U4 MCP73831-2-OT, U5 MS5637, U6 W25N01GVZEIG, U7 ICM-20948, U8 L96-M33, U9 AP22804, Y1 8MHz

Commit message: all components placed, initial board art
Parts:
- gave numbers to parts that had none: 2
Other:
- moved on the sheet: C34, C35, C36, C37, C38, C39, C40, C41

Commit message: final checkouts
Parts:
- removed J10: CELL, Connector_JST:JST_SH_BM03B-SRSS-TB_1x03-1MP_P1.00mm_Vertical, symbol Connector_Generic:Conn_01x03
- removed J8: NCP_COM, Connector_PinHeader_1.27mm:PinHeader_1x07_P1.27mm_Vertical, symbol Connector_Generic:Conn_01x07
- removed U10: AP2120N-1.8, Package_TO_SOT_SMD:SOT-23, symbol Regulator_Linear:AP2127N-1.8
- removed U11: FXLA0104, atlas:UMLP-12, symbol glider:FXLA0104
- removed U3: MCP1812, Package_TO_SOT_SMD:SOT-23, symbol atlas:MCP1811B
- added C43, C44: 4.7u, Capacitor_SMD:C_0805_2012Metric, symbol Device:C_Small
- added J8: NCP_COM, Connector_PinHeader_2.54mm:PinHeader_1x08_P2.54mm_Vertical, symbol Connector_Generic:Conn_01x08
- added LS1: PKLCS1212E40A1-R1, atlas:PKLCS1212, symbol Device:Speaker
- added Q2, Q3: 2N7002E, Package_TO_SOT_SMD:SOT-23, symbol Device:Q_NMOS_GSD
- added R30: 100k, Resistor_SMD:R_0603_1608Metric, symbol Device:R_Small
- added R31: 1k, Resistor_SMD:R_0603_1608Metric, symbol Device:R_Small
- added U10: MIC5501-3.0YM5, Package_TO_SOT_SMD:SOT-23-5, symbol Regulator_Linear:MIC5501-3.0YM5
- added U11: NTB0104, atlas:WQFN-14-1EP_2.5x3mm_P0.5mm_EP1.45x1.00mm, symbol glider:NTB0104
- added U3: MIC5504-1.8YM5, Package_TO_SOT_SMD:SOT-23-5, symbol Regulator_Linear:MIC5504-1.8YM5
- C15: value C_Small -> 0.1u
- C22, C31, C32, C34, C35, C36, C37, C38, C39, C40, C41: value 22u -> 10u
- D7: value NAV_STAT_1 -> NCP_STAT1
- D9: value NAV_STAT_0 -> NCP_STAT0
- J20: value Conn_01x02 -> CELL; footprint Connector_PinSocket_2.54mm:PinSocket_1x02_P2.54mm_Vertical -> Connector_PinSocket_2.54mm:PinSocket_1x03_P2.54mm_Vertical; symbol Connector_Generic:Conn_01x02 -> Connector_Generic:Conn_01x03
- J3: footprint Connector_PinHeader_1.27mm:PinHeader_1x07_P1.27mm_Vertical -> Connector_PinHeader_1.27mm:PinHeader_1x08_P1.27mm_Vertical; symbol Connector_Generic:Conn_01x07 -> Connector_Generic:Conn_01x08
- Q1: value Q_PMOS_DGS -> DMP1045UQ; symbol Device:Q_PMOS_DGS -> Device:Q_PMOS_GSD
- R1: value 2k -> 10k
- R13, R14: footprint Resistor_SMD:R_0603_1608Metric -> Resistor_SMD:R_0402_1005Metric
- R25: value 10k -> 100k
- SW1, SW2, SW3, SW4: footprint Button_Switch_SMD:SW_SPST_B3U-1000P -> Button_Switch_SMD:SW_SPST_PTS810
Connections:
- net labels added: BUZZER_TIM2_CH4
- net labels removed: GPS_PPS_LED
- wire segments 588 -> 620
Other:
- moved on the sheet: C11, C12, C22, C24, C26, C34, C35, C36, C37, C38, C39, C40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

Commit message: removed bt module again, shrunk board
Parts:
- removed AE1: Antenna_Shield, Connector_Coaxial:U.FL_Hirose_U.FL-R-SMT-1_Vertical, symbol Device:Antenna_Shield
- removed C14, C2, C42: 0.1u, Capacitor_SMD:C_0402_1005Metric, symbol Device:C_Small
- removed D7: NCP_STAT1, LED_SMD:LED_0603_1608Metric, symbol Device:LED_Small_ALT
- removed D8: NAV_STAT_2, LED_SMD:LED_0603_1608Metric, symbol Device:LED_Small_ALT
- removed D9: NCP_STAT0, LED_SMD:LED_0603_1608Metric, symbol Device:LED_Small_ALT
- removed J19: Micro_SD_Card, Connector_Card:microSD_HC_Hirose_DM3D-SF, symbol Connector:Micro_SD_Card
- removed J3: NCP_EXT, Connector_PinHeader_1.27mm:PinHeader_1x08_P1.27mm_Vertical, symbol Connector_Generic:Conn_01x08
- removed J5: DEBUG_NCP, Connector_PinHeader_1.27mm:PinHeader_2x05_P1.27mm_Vertical_SMD, symbol atlas:Conn_ARM_JTAG_SWD_10
- removed L2: 47n, Inductor_SMD:L_0402_1005Metric, symbol Device:L_Small
- removed R10, R29, R9: 1k, Resistor_SMD:R_0603_1608Metric, symbol Device:R_Small
- removed R13, R14, R21: 0, Resistor_SMD:R_0402_1005Metric, symbol Device:R_Small
- removed R16, R19: 100k, Resistor_SMD:R_0603_1608Metric, symbol Device:R_Small
- removed R22: 10, Resistor_SMD:R_0603_1608Metric, symbol Device:R_Small
- removed SW3: NCP_NRST, Button_Switch_SMD:SW_SPST_PTS810, symbol Switch:SW_SPST
- removed SW4: NCP_USER, Button_Switch_SMD:SW_SPST_PTS810, symbol Switch:SW_SPST
- removed U1: BGM220P, atlas:BGM220P, symbol atlas:BGM220P
- removed U9: AP22804, Package_DFN_QFN:DFN-6-1EP_2x2mm_P0.65mm_EP1x1.6mm, symbol atlas:AP22804
- added H4: MountingHole_Pad, MountingHole:MountingHole_2.5mm_Pad_Via, symbol Mechanical:MountingHole_Pad
- added J10: DM3CS-SF, HRS_DM3CS-SF, symbol DM3CS-SF:DM3CS-SF
- J8: footprint Connector_PinHeader_2.54mm:PinHeader_1x08_P2.54mm_Vertical -> Connector_PinHeader_2.54mm:PinHeader_1x05_P2.54mm_Vertical; symbol Connector_Generic:Conn_01x08 -> Connector_Generic:Conn_01x05
Connections:
- net GND: now also H4.1, J10.6 (VSS), J10.S1 (GND), J10.S2 (GND), J10.S3 (GND), J10.S5 (GND)
- net IMU_SPI2_MISO: now also J10.7 (DAT0)
- net IMU_SPI2_MOSI: now also J10.3 (CMD)
- net IMU_SPI2_SCK: now also J10.5 (CLK)
- net SD_NCS: now also J10.2 (CD/DAT3)
- net VDD_MCU: now also U?1.5 (XSHUT), J10.4 (VDD)
- net at D1.1 (K): now also U4.1 (STAT); no longer R2.2
- net at C13.1, C8.1, D3.2 (A)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: now also R2.2; no longer D1.2 (A)
- net at R2.1: now also D1.2 (A); no longer U4.1 (STAT)
- net GPS_I2C_SCL: no longer names the net of U8.6 (I2C_SCL)
- net GPS_I2C_SDA: no longer names the net of U8.3 (I2C_SDA)
- net NCP_COM0 renamed RADIO_USART3_TX
- net NCP_COM1 renamed RADIO_USART3_RX
- net NCP_COM2 renamed RADIO_SET
- net NCP_COM3: no longer names the net of U2.35 (PB13)
- net NCP_COM3: no longer J8.6 (Pin_6)
- net NCP_COM4: no longer names the net of U2.36 (PB14)
- net NCP_COM4: no longer J8.7 (Pin_7)
- net NCP_COM5: no longer names the net of U2.37 (PB15)
- net NCP_COM5: no longer J8.8 (Pin_8)
- net TOF_EN: no longer names the net of U2.55 (PD2)
- net TOF_EN: no longer U?1.5 (XSHUT)
- no-connect marks 14 -> 12
Other:
- moved on the sheet: C15, D1, R2, U6

Commit message: reved layout complete, silkscreen todo
Parts:
- removed C6: 0.1u, Capacitor_SMD:C_0402_1005Metric, symbol Device:C_Small
- removed U?1: VL53L1CXV0FY, atlas:LGA-12-3.7x2.1mm, symbol glider:VL53L1CXV0FY
- added C14, C2: 10u, Capacitor_SMD:C_1206_3216Metric, symbol Device:C_Small
- added J3: HPS_A, Resistor_SMD:R_2816_7142Metric_Pad3.20x4.45mm_HandSolder, symbol Connector_Generic:Conn_01x02
- added JP2: HPS_CELL_V, Jumper:SolderJumper-2_P1.3mm_Open_TrianglePad1.0x1.5mm, symbol Device:Jumper_NO_Small
- added Q4: DMT6008LFG, atlas:Diodes_PowerDI3333-8, symbol Device:Q_NMOS_GDS
- added R13: 0.1, Resistor_SMD:R_1210_3225Metric, symbol Device:R_Small
- C19, C20: value 0.1u -> 10u; footprint Capacitor_SMD:C_0402_1005Metric -> Capacitor_SMD:C_1206_3216Metric
- J1: footprint Connector_PinHeader_1.27mm:PinHeader_1x03_P1.27mm_Vertical -> Connector_PinHeader_2.54mm:PinHeader_1x05_P2.54mm_Vertical; symbol Connector_Generic:Conn_01x03 -> Connector_Generic:Conn_01x05
- J12: footprint Connector_PinHeader_1.27mm:PinHeader_1x03_P1.27mm_Vertical -> Connector_PinHeader_1.27mm:PinHeader_1x04_P1.27mm_Vertical; symbol Connector_Generic:Conn_01x03 -> Connector_Generic:Conn_01x04
- Y1: symbol Device:Crystal -> Device:Crystal_GND24
Connections:
- net CELL_POS: now also JP2.1
- net GND: now also J1.2 (Pin_2), J12.2 (Pin_2), Y1.2, Y1.4, C14.2, C2.2, R13.2; no longer J1.1 (Pin_1)
- net GPS_EXTINT: now also U2.4 (PC15/OSC32_O); no longer U2.3 (PC14/OSC32_I)
- net GPS_FIX: no longer U2.4 (PC15/OSC32_O)
- net GPS_FORCEON: now also U2.3 (PC14/OSC32_I); no longer U2.2 (PC13)
- net GPS_RESET: now also U2.2 (PC13); no longer U2.62 (PB9)
- net IMU_INT: now also U2.62 (PB9); no longer U2.58 (PB5)
- net IMU_SPI2_MOSI: now also U2.58 (PB5); no longer U2.54 (PC12)
- net IO_TIM8_CH1: now also J11.2 (Pin_2); no longer J15.2 (Pin_2)
- net IO_TIM8_CH2: now also J13.2 (Pin_2); no longer J14.2 (Pin_2)
- net IO_TIM8_CH3: now also J14.2 (Pin_2); no longer J13.2 (Pin_2)
- net IO_TIM8_CH4: now also J15.2 (Pin_2); no longer J11.2 (Pin_2)
- net RADIO_SET: now also U2.44 (PA10); no longer U2.34 (PB12)
- net RADIO_USART3_RX: now also U2.55 (PD2); no longer U2.33 (PB11)
- net RADIO_USART3_TX: now also U2.54 (PC12); no longer U2.30 (PB10)
- net SENSOR_I2C_SDA: now also J1.4 (Pin_4); no longer J1.2 (Pin_2)
- net VDD_MCU: now also J1.1 (Pin_1); no longer C19.1, C20.1
- net OPAMP4_CELL_VS: now reaches U2.35 (PB13)
- net OPAMP4_CELL_VS: now also R24.2, R25.1
- net OPAMP2_CELL_IS: now reaches U2.36 (PB14)
- net OPAMP2_CELL_IS: now also J20.3 (Pin_3), R4.1
- net ADC2_IN15_CELL_TS: now reaches U2.37 (PB15)
- net ADC2_IN15_CELL_TS: now also J20.2 (Pin_2), R28.1, R7.2
- net at C4.1, Y1.1: now also U2.5 (PF0/OSC_I); no longer U2.6 (PF1/OSC_O)
- removed net ADC1_IN1_CELL_TS: J20.2 (Pin_2), R28.1, R7.2, U2.12 (PA0)
- net BUZZER_TIM2_CH4 renamed BUZZER_TIM3_CH2
- net BUZZER_TIM3_CH2: now also U2.18 (PA4); no longer U2.44 (PA10)
- net IO_TIM2_CH1 renamed IO_0
- net IO_0: now also J12.4 (Pin_4); no longer J12.3 (Pin_3)
- net IO_TIM3_CH2 renamed IO_TIM1_CH4
- net IO_TIM1_CH4: now also U2.11 (PC3); no longer U2.18 (PA4)
- removed net OPAMP3_CELL_IS: J20.3 (Pin_3), R4.1, U2.13 (PA1)
- net OPAMP3_VINM0 renamed IO_1
- net IO_1: now also J12.3 (Pin_3); no longer J12.2 (Pin_2)
- removed net OPAMP5_CELL_VS: R24.2, R25.1, U2.11 (PC3)
- new net: C3.1, U2.6 (PF1/OSC_O), Y1.3
- new net: C14.1, C19.1, C2.1, C20.1, J3.1 (Pin_1), JP2.2
- new net: J3.2 (Pin_2), Q4.2 (D)
- new net HPS_A_OPAMP3_CS: Q4.3 (S), R13.1, U2.34 (PB12)
- new net HPS_A_TIM3_CH2: Q4.1 (G), U2.33 (PB11)
- new net HPS_B_OPAMP6_CS: U2.13 (PA1)
- new net HPS_B_TIM2_CH1: U2.12 (PA0)
- new net I2C_EXT_INT: J1.5 (Pin_5), U2.30 (PB10)
Other:
- moved on the sheet: C3, C4, J7, J8, J9

Commit message: submitted to jlc
Parts:
- added D7: SD1206T040S2R0, Diode_SMD:D_SOD-123, symbol Device:D_Schottky_Small_ALT
- added D8: USB_PWR, LED_SMD:LED_0603_1608Metric, symbol Device:LED_Small_ALT
- added JP2: HPS_CELL_V, Jumper:SolderJumper-2_P1.3mm_Open_TrianglePad1.0x1.5mm, symbol Device:Jumper_NO_Small
- added N1: Bottom Graphic, atlas:boardartswift, symbol Mechanical:Housing
- added R24: 100k, Resistor_SMD:R_0603_1608Metric, symbol Device:R_Small
- added R25: 1k, Resistor_SMD:R_0603_1608Metric, symbol Device:R_Small
- added TP1: VREFBUF, TestPoint:TestPoint_THTPad_D1.0mm_Drill0.5mm, symbol Connector:TestPoint
- added TP2: VCC_SYS, TestPoint:TestPoint_THTPad_D1.0mm_Drill0.5mm, symbol Connector:TestPoint
- added TP3: VDD_MCU, TestPoint:TestPoint_THTPad_D1.0mm_Drill0.5mm, symbol Connector:TestPoint
- added TP4: VDD_IMU, TestPoint:TestPoint_THTPad_D1.0mm_Drill0.5mm, symbol Connector:TestPoint
- D2: renamed from D3; value D_Schottky -> SD1206T040S2R0
- renumbered C19 to C1, C20 to C10, C16 to C11, C18 to C12, C24 to C13, C21 to C14, C22 to C15, C8 to C16, C13 to C17, C25 to C18, C26 to C19, C1 to C2, C27 to C20, C28 to C21, C29 to C22, C30 to C23, C17 to C24, C31 to C25, C23 to C26, C32 to C27, C33 to C28, C44 to C29, C4 to C3, C10 to C30, C15 to C31, C11 to C32, C12 to C33, C43 to C34, C34 to C35, C35 to C36, C36 to C37, C37 to C38, C38 to C39, C3 to C4, C39 to C40, C40 to C41, C41 to C42, C2 to C5, C5 to C6, C14 to C8, D2 to D3, J3 to J1, J16 to J10, J17 to J11, J18 to J12, J6 to J13, J1 to J14, J12 to J15, J7 to J16, J8 to J17, J9 to J18, J4 to J2, J20 to J3, J2 to J4, J10 to J5, J11 to J6, J13 to J7, J14 to J8, J15 to J9, JP2 to JP1, L3 to L2, Q4 to Q1, Q1 to Q2, Q2 to Q3, Q3 to Q4, R13 to R1, R27 to R10, R30 to R11, R18 to R12, R24 to R13, R25 to R14, R31 to R15, R7 to R16, R28 to R17, R6 to R18, R8 to R19, R4 to R2, R5 to R20, R15 to R21, R17 to R22, R20 to R23, R23 to R3, R1 to R4, R11 to R5, R12 to R6, R2 to R7, R3 to R8, R26 to R9, SW2 to SW1, SW1 to SW2, U2 to U1, U6 to U10, U3 to U2, U11 to U3, U5 to U4, U12 to U5, U4 to U6, U10 to U9
Connections:
- net HPS_B_TIM2_CH1 is gone; now on net GPS_FIX: U1.12 (PA0)
- net CELL_POS: now also JP2.1
- net GND: now also D8.1 (K), R24.1
- net VDD_IMU: now also TP4.1
- net VDD_MCU: now also TP3.1; no longer U3.8 (OE)
- net VDD_SYS: now also TP2.1
- net VREFBUF_OUT: now also TP1.1
- net VCC_USB: now reaches C16.1, C17.1, D2.2 (A), F1.1, Q2.1 (G), R4.2, R7.2, R8.2, U6.4 (VDD)
- net VCC_USB: now also R25.1
- net at C1.1, C10.1, C5.1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: now also D7.1 (K), JP2.2
- net at J1.2 (Pin_2), Q1.2 (D): now also D7.2 (A)
- net HPS_B_OPAMP6_CS renamed IMU_SPI_LS_EN
- net IMU_SPI_LS_EN: now also U3.8 (OE), R24.2
- net IMU_SPI2_MISO renamed IMU_SPI3_MISO
- net IMU_SPI2_MOSI renamed IMU_SPI3_MOSI
- net IMU_SPI2_SCK renamed IMU_SPI3_SCK
- new net: D8.2 (A), R25.2
Other:
- moved on the sheet: C1, C10, C31, C5, C8, J1, JP1, Q1, R1, U10
